File: rxfilter.kicad_sch (KiCad schematic)
At the start: 13 parts

Commit message: Fix capacitor values
Parts:
- C?: value 0.1u -> 0.1uF
Changed lines of the file:
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@@
 		(shape input)
 		(at 207.01 93.98 0)
-		(fields_autoplaced yes)
 		(effects
 			(font
@@
 		(shape input)
 		(at 207.01 86.36 0)
-		(fields_autoplaced yes)
 		(effects
 			(font
@@
 		(shape input)
 		(at 82.55 87.63 180)
-		(fields_autoplaced yes)
 		(effects
 			(font
@@
 		(shape input)
 		(at 207.01 90.17 0)
-		(fields_autoplaced yes)
 		(effects
 			(font
@@
 			)
 		)
-		(property "Value" "0.1u"
+		(property "Value" "0.1uF"
 			(at 181.864 74.676 90)
 			(effects

Commit message: Fill up mouser part numbers
Parts:
- C?: MouserPN (none) -> 581-KGM05AR71C104KN
- C? (x2): MouserPN (none) -> 187-CL05C101JC51PNC
- D?: MouserPN (none) -> 621-BAT54WS-F
- FB?: MouserPN (none) -> 81-BLM15AG102SZ1D
- U?: MouserPN (none) -> 926-LMV7271MG/NOPB
Changed lines of the file:
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@@
+			)
+		)
+		(property "MouserPN" "581-KGM05AR71C104KN"
+			(at 181.61 80.01 0)
+			(effects
+				(font
+					(size 1.27 1.27)
+				)
+				(hide yes)
+			)
+		)
+		(property "Quantity" ""
+			(at 181.61 80.01 0)
+			(effects
+				(font
+					(size 1.27 1.27)
+				)
+				(hide yes)
 			)
 		)
@@
 			)
 		)
+		(property "MouserPN" "187-CL05C101JC51PNC"
+			(at 123.19 107.95 0)
+			(effects
+				(font
+					(size 1.27 1.27)
+				)
+				(hide yes)
+			)
+		)
+		(property "Quantity" ""
+			(at 123.19 107.95 0)
+			(effects
+				(font
+					(size 1.27 1.27)
+				)
+				(hide yes)
+			)
+		)
 		(pin "1"
 		)
@@
 			)
 		)
+		(property "MouserPN" "621-BAT54WS-F"
+			(at 105.41 87.63 0)
+			(effects
+				(font
+					(size 1.27 1.27)
+				)
+				(hide yes)
+			)
+		)
+		(property "Quantity" ""
+			(at 105.41 87.63 0)
+			(effects
+				(font
+					(size 1.27 1.27)
+				)
+				(hide yes)
+			)
+		)
 		(pin "1"
 		)
@@
 		)
 		(property "Description" ""
+			(at 191.77 90.17 0)
+			(effects
+				(font
+					(size 1.27 1.27)
+				)
+				(hide yes)
+			)
+		)
+		(property "MouserPN" ""
+			(at 191.77 90.17 0)
+			(effects
+				(font
+					(size 1.27 1.27)
+				)
+				(hide yes)
+			)
+		)
+		(property "Quantity" ""
 			(at 191.77 90.17 0)
 			(effects
@@
 			)
 		)
+		(property "MouserPN" "187-CL05C101JC51PNC"
+			(at 132.08 87.63 0)
+			(effects
+				(font
+					(size 1.27 1.27)
+				)
+				(hide yes)
+			)
+		)
+		(property "Quantity" ""
+			(at 132.08 87.63 0)
+			(effects
+				(font
+					(size 1.27 1.27)
+				)
+				(hide yes)
+			)
+		)
 		(pin "1"
 		)
@@
 			)
 		)
+		(property "MouserPN" "81-BLM15AG102SZ1D"
+			(at 176.53 64.77 0)
+			(effects
+				(font
+					(size 1.27 1.27)
+				)
+				(hide yes)
+			)
+		)
+		(property "Quantity" ""
+			(at 176.53 64.77 0)
+			(effects
+				(font
+					(size 1.27 1.27)
+				)
+				(hide yes)
+			)
+		)
 		(pin "1"
 		)
@@
 			)
 		)
+		(property "MouserPN" "926-LMV7271MG/NOPB"
+			(at 179.07 90.17 0)
+			(effects
+				(font
+					(size 1.27 1.27)
+				)
+				(hide yes)
+			)
+		)
+		(property "Quantity" ""
+			(at 179.07 90.17 0)
+			(effects
+				(font
+					(size 1.27 1.27)
+				)
+				(hide yes)
+			)
+		)
 		(pin "1"
 		)
@@
 			)
 		)
+		(property "MouserPN" ""
+			(at 160.02 107.95 0)
+			(effects
+				(font
+					(size 1.27 1.27)
+				)
+				(hide yes)
+			)
+		)
+		(property "Quantity" ""
+			(at 160.02 107.95 0)
+			(effects
+				(font
+					(size 1.27 1.27)
+				)
+				(hide yes)
+			)
+		)
 		(pin "1"
 		)
@@
 			)
 		)
+		(property "MouserPN" ""
+			(at 90.17 87.63 0)
+			(effects
+				(font
+					(size 1.27 1.27)
+				)
+				(hide yes)
+			)
+		)
+		(property "Quantity" ""
+			(at 90.17 87.63 0)
+			(effects
+				(font
+					(size 1.27 1.27)
+				)
+				(hide yes)
+			)
+		)
 		(pin "1"
 		)
@@
 			)
 		)
+		(property "MouserPN" ""
+			(at 160.02 78.74 0)
+			(effects
+				(font
+					(size 1.27 1.27)
+				)
+				(hide yes)
+			)
+		)
+		(property "Quantity" ""
+			(at 160.02 78.74 0)
+			(effects
+				(font
+					(size 1.27 1.27)
+				)
+				(hide yes)
+			)
+		)
 		(pin "1"
 		)
@@
 			)
 		)
+		(property "MouserPN" ""
+			(at 142.24 78.74 0)
+			(effects
+				(font
+					(size 1.27 1.27)
+				)
+				(hide yes)
+			)
+		)
+		(property "Quantity" ""
+			(at 142.24 78.74 0)
+			(effects
+				(font
+					(size 1.27 1.27)
+				)
+				(hide yes)
+			)
+		)
 		(pin "1"
 		)
@@
 			)
 		)
+		(property "MouserPN" ""
+			(at 142.24 107.95 0)
+			(effects
+				(font
+					(size 1.27 1.27)
+				)
+				(hide yes)
+			)
+		)
+		(property "Quantity" ""
+			(at 142.24 107.95 0)
+			(effects
+				(font
+					(size 1.27 1.27)
+				)
+				(hide yes)
+			)
+		)
 		(pin "1"
 		)
@@
 			(at 113.03 102.87 0)
 			(effects
+				(font
+					(size 1.27 1.27)
+				)
+				(hide yes)
+			)
+		)
+		(property "MouserPN" ""
+			(at 113.03 102.87 0)
+			(effects
+				(font
+					(size 1.27 1.27)
+				)
+				(hide yes)
+			)
+		)
+		(property "Quantity" ""
+			(at 113.03 102.87 0)
+			(effects

Commit message: Finish BOM components filling
Parts:
- R?: MouserPN (none) -> 594-MCS04020C4702FE0
- R?: MouserPN (none) -> 71-CRCW040210K0FKEDC
- R? (x2): MouserPN (none) -> 652-CR0402FX5232GLF
- R? (x2): MouserPN (none) -> 603-RC0402FR-7D100KL
- TP?: now left out of the parts list
Changed lines of the file:
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@@
 		(unit 1)
 		(exclude_from_sim no)
-		(in_bom yes)
+		(in_bom no)
 		(on_board yes)
 		(dnp no)
@@
 			)
 		)
-		(property "MouserPN" ""
+		(property "MouserPN" "594-MCS04020C4702FE0"
 			(at 160.02 107.95 0)
 			(effects
@@
 			)
 		)
-		(property "MouserPN" ""
+		(property "MouserPN" "71-CRCW040210K0FKEDC"
 			(at 90.17 87.63 0)
 			(effects
@@
 			)
 		)
-		(property "MouserPN" ""
+		(property "MouserPN" "652-CR0402FX5232GLF"
 			(at 160.02 78.74 0)
 			(effects
@@
 			)
 		)
-		(property "MouserPN" ""
+		(property "MouserPN" "603-RC0402FR-7D100KL"
 			(at 142.24 78.74 0)
 			(effects
@@
 			)
 		)
-		(property "MouserPN" ""
+		(property "MouserPN" "603-RC0402FR-7D100KL"
 			(at 142.24 107.95 0)
 			(effects
@@
 			)
 		)
-		(property "MouserPN" ""
+		(property "MouserPN" "652-CR0402FX5232GLF"
 			(at 113.03 102.87 0)
 			(effects
