File: power.kicad_sch (KiCad schematic)
At the start: 62 parts, among them Q2 NTR5105PT1G, Q5 NX138BKWX, Q9 BC846BS

Commit message: Fix BOM
Parts:
- C? (x4): MouserPN 581-1210YG474ZAT2A -> 80-C1210C476M4P7210
- C?: MouserPN 581-02013A100J -> 581-06033D475KAT2A
Changed lines of the file:
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@@
 			)
 		)
-		(property "MouserPN" "581-1210YG474ZAT2A "
+		(property "MouserPN" "80-C1210C476M4P7210"
 			(at 215.9 100.33 0)
 			(effects
@@
 			)
 		)
-		(property "MouserPN" "581-1210YG474ZAT2A "
+		(property "MouserPN" "80-C1210C476M4P7210"
 			(at 170.18 100.33 0)
 			(effects
@@
 			)
 		)
-		(property "MouserPN" "581-1210YG474ZAT2A "
+		(property "MouserPN" "80-C1210C476M4P7210"
 			(at 185.42 100.33 0)
 			(effects
@@
 			)
 		)
-		(property "MouserPN" "581-1210YG474ZAT2A "
+		(property "MouserPN" "80-C1210C476M4P7210"
 			(at 200.66 100.33 0)
 			(effects
@@
 			)
 		)
-		(property "MouserPN" "581-02013A100J"
+		(property "MouserPN" "581-06033D475KAT2A"
 			(at 184.15 66.04 0)
 			(effects
